Commit message: added in lidar

File: src/aug_2024/description/urdf/aug_2024.xacro (robot description, xacro)
@@ -31,4 +31,10 @@
     </inertial>
   </link>
+<link name="base_footprint"/>
+<joint name="base_joint" type="fixed">
+  <parent link="base_footprint"/>
+  <child link="base_link"/>
+  <origin xyz="0 0 0.1016" rpy="0 0 0"/>
+</joint>
 <link name="chassis_link">
   <visual>
@@ -272,4 +278,62 @@
 <gazebo reference="left_caster_wheel_joint">
   <implicitSpringDamper>1</implicitSpringDamper>
+</gazebo>
+<!--LIDAR-->
+<link name="lidar_link">
+  <visual>
+    <geometry>
+      <cylinder radius="0.05" length="0.04"/>
+    </geometry>
+    <material name="black"/>
+  </visual>
+  <collision>
+    <geometry>
+      <cylinder radius="0.05" length="0.04"/>
+    </geometry>
+  </collision>
+  <inertial>
+    <mass value="0.1"/>
+    <inertia ixx="0.000033" ixy="0.0" ixz="0.0" iyy="0.000033" iyz="0.0" izz="0.00006"/>
+  </inertial>
+</link>
+<joint name="lidar_joint" type="fixed">
+  <parent link="chassis_link"/>
+  <child link="lidar_link"/>
+  <origin xyz="0 0 0.1" rpy="0 0 0"/>
+</joint>
+<gazebo reference="lidar_link">
+  <sensor type="gpu_ray" name="lidar">
+    <pose>0 0 0 0 0 0</pose>
+    <visualize>false</visualize>
+    <update_rate>10</update_rate>
+    <ray>
+      <scan>
+        <horizontal>
+          <samples>360</samples>
+          <resolution>1</resolution>
+          <min_angle>-3.14159</min_angle>
+          <max_angle>3.14159</max_angle>
+        </horizontal>
+      </scan>
+      <range>
+        <min>0.3</min>
+        <max>12.0</max>
+        <resolution>0.01</resolution>
+      </range>
+      <noise>
+        <type>gaussian</type>
+        <mean>0.0</mean>
+        <stddev>0.01</stddev>
+      </noise>
+    </ray>
+    <plugin name="gazebo_ros_lidar_controller" filename="libgazebo_ros_ray_sensor.so">
+      <ros>
+        <namespace>/</namespace>
+        <remapping>~/out:=scan</remapping>
+      </ros>
+      <output_type>sensor_msgs/msg/LaserScan</output_type>
+      <frame_name>lidar_link</frame_name>
+    </plugin>
+  </sensor>
 </gazebo>
 <!--ROS CONTROL SECTION-->
