Commit message: everything works so-so

File: install/aug_2024/share/aug_2024/description/urdf/aug_2024.urdf (robot description, URDF)
Before this commit: robot aug_2024_bot, 4 links, 3 joints
Links:
- added link lidar_link, mass 0.1; collision cylinder length=0.04 radius=0.05; visual cylinder length=0.04 radius=0.05
- added link rear_left_wheel_link; collision cylinder length=0.04 radius=0.10; visual cylinder length=0.04 radius=0.10
- added link rear_right_wheel_link; collision cylinder length=0.04 radius=0.10; visual cylinder length=0.04 radius=0.10
- link base_link: geometry collision box size=0.42 0.31 0.18; visual box size=0.42 0.31 0.18
- link front_caster: geometry collision sphere radius=.06; visual sphere radius=.06
Joints:
- added joint lidar_joint: type fixed, parent base_link, child lidar_link, origin xyz=0 0 0.1 rpy=0 0 0
- added joint rear_left_wheel_joint: type continuous, parent base_link, child rear_left_wheel_link, origin xyz=-0.12 .18 -.05 rpy=0 0 0, axis 0 1 0
- added joint rear_right_wheel_joint: type continuous, parent base_link, child rear_right_wheel_link, origin xyz=-0.12 -.18 -.05 rpy=0 0 0, axis 0 1 0
- joint base_joint: child base_footprint -> base_link; origin xyz=0.0 0.0 ${-(wheel_radius+wheel_zoff)} rpy=0 0 0 -> xyz=0.0 0.0 0.2 rpy=0 0 0; parent base_link -> base_footprint
- joint caster_joint: origin xyz=${caster_xoff} 0.0 ${-(base_height/2)} rpy=0 0 0 -> xyz=0.14 0.0 -.09 rpy=0 0 0

Commit message: 1-20-25_all works

File: install/aug_2024/share/aug_2024/description/urdf/aug_2024.urdf (robot description, URDF)
Before this commit: robot aug_2024_bot, 7 links, 6 joints
Links:
- removed link front_caster
- added link left_caster_pivot_link; collision cylinder length=0.02 radius=0.02; visual cylinder length=0.02 radius=0.02
- added link left_wheel_link; collision cylinder length=0.02 radius=0.04; visual cylinder length=0.02 radius=0.04
- added link right_caster_pivot_link; collision cylinder length=0.02 radius=0.02; visual cylinder length=0.02 radius=0.02
- added link right_wheel_link; collision cylinder length=0.02 radius=0.04; visual cylinder length=0.02 radius=0.04
- link base_link: geometry collision box size=0.32 0.21 0.18; visual box size=0.32 0.21 0.18
Joints:
- removed joint caster_joint
- added joint left_caster_pivot_joint: type continuous, parent base_link, child left_caster_pivot_link, origin xyz=.2 .2 -0.06 rpy=0 0 0, axis 0 0 1
- added joint left_wheel_joint: type continuous, parent left_caster_pivot_link, child left_wheel_link, origin xyz=-.050 0 -0.05 rpy=1.57079632679 0 0, axis 0 0 1
- added joint right_caster_pivot_joint: type continuous, parent base_link, child right_caster_pivot_link, origin xyz=.2 -.2 -0.06 rpy=0 0 0, axis 0 0 1
- added joint right_wheel_joint: type continuous, parent right_caster_pivot_link, child right_wheel_link, origin xyz=-.050 0 -0.05 rpy=1.57079632679 0 0, axis 0 0 1
