Commit message: 2-20-25

File: install/aug_2024/share/aug_2024/description/urdf/aug_2024-nocaster.urdf (robot description, URDF)
Before this commit: robot aug_2024_bot, 7 links, 6 joints
Links:
- added link camera_link; visual box size=0.05 0.05 0.05
- link rear_left_wheel_link: geometry collision cylinder length=0.04 radius=0.10; visual box size=0.04 0.01 0.19
- link rear_right_wheel_link: geometry collision cylinder length=0.04 radius=0.10; visual box size=0.04 0.01 0.19
Joints:
- added joint camera_joint: type fixed, parent base_link, child camera_link, origin xyz=0.1 0 0.2 rpy=0 0 0
- joint base_joint: origin xyz=0.0 0.0 0.2 rpy=0 0 0 -> xyz=0.0 0.0 0.15 rpy=0 0 0
- joint caster_joint: axis (none) -> 0 0 1; origin xyz=0.14 0.0 -.09 rpy=0 0 0 -> xyz=-0.14 0.0 -.07 rpy=0 0 0
- joint rear_left_wheel_joint: origin xyz=-0.12 .18 -.05 rpy=0 0 0 -> xyz=0.05 .25 -.03 rpy=0 0 0
- joint rear_right_wheel_joint: origin xyz=-0.12 -.18 -.05 rpy=0 0 0 -> xyz=0.05 -.25 -.03 rpy=0 0 0

File: src/aug_2024/description/urdf/aug_2024-nocaster.urdf (robot description, URDF)
Before this commit: robot aug_2024_bot, 7 links, 6 joints
Links:
- added link camera_link; visual box size=0.05 0.05 0.05
- link rear_left_wheel_link: geometry collision cylinder length=0.04 radius=0.10; visual box size=0.04 0.01 0.19
- link rear_right_wheel_link: geometry collision cylinder length=0.04 radius=0.10; visual box size=0.04 0.01 0.19
Joints:
- added joint camera_joint: type fixed, parent base_link, child camera_link, origin xyz=0.1 0 0.2 rpy=0 0 0
- joint base_joint: origin xyz=0.0 0.0 0.2 rpy=0 0 0 -> xyz=0.0 0.0 0.15 rpy=0 0 0
- joint caster_joint: axis (none) -> 0 0 1; origin xyz=0.14 0.0 -.09 rpy=0 0 0 -> xyz=-0.14 0.0 -.07 rpy=0 0 0
- joint rear_left_wheel_joint: axis 0 -1 0 -> 0 1 0; origin xyz=-0.12 .18 -.05 rpy=0 0 0 -> xyz=0.05 .25 -.03 rpy=0 0 0
- joint rear_right_wheel_joint: axis 0 -1 0 -> 0 1 0; origin xyz=-0.12 -.18 -.05 rpy=0 0 0 -> xyz=0.05 -.25 -.03 rpy=0 0 0

Commit message: working on desktop ready for rospi

File: install/aug_2024/share/aug_2024/description/urdf/aug_2024-nocaster.urdf (robot description, URDF)
Before this commit: robot aug_2024_bot, 7 links, 6 joints
Joints:
- joint rear_left_wheel_joint: axis 0 1 0 -> 0 -1 0
- joint rear_right_wheel_joint: axis 0 1 0 -> 0 -1 0

Commit message: added in video support

File: install/aug_2024/share/aug_2024/description/urdf/aug_2024-nocaster.urdf (robot description, URDF)
Before this commit: robot aug_2024_bot, 7 links, 6 joints
Links:
- added link camera_link, mass 0.1; collision box size=0.010 0.03 0.03; visual box size=0.010 0.03 0.03
- added link camera_optical_link
Joints:
- added joint camera_joint: type fixed, parent base_link, child camera_link, origin xyz=0.2 0 0.075 rpy=0 0 0
- added joint camera_optical_joint: type fixed, parent camera_link, child camera_optical_link, origin xyz=0 0 0 rpy=-1.57079632679 0 -1.57079632679
